Commit message: change to big spoon

File: assets/urdf/spoon/urdf/spoon.urdf (robot description, URDF)
Before this commit: robot spoon, 1 links, 0 joints
Links:
- link base_link: mass 0.032987 -> 0.079407

Commit message: update spoon

File: assets/urdf/spoon/urdf/spoon.urdf (robot description, URDF)
Before this commit: robot spoon, 1 links, 0 joints
Links:
- link base_link: mass 0.079407 -> 1.026

Commit message: change spoon to normal spoon

File: assets/urdf/spoon/urdf/spoon.urdf (robot description, URDF)
Before this commit: robot spoon, 1 links, 0 joints
Links:
- link base_link: mass 1.026 -> 0.032987
