Commit message: fix shelf

File: assets/urdf/shelf/urdf/shelf.urdf (robot description, URDF)
Before this commit: robot shelf, 1 links, 0 joints
Links:
- link base_link: geometry collision box size=0.011 0.08324 0.11; collision box size=0.011 0.08324 0.11

Commit message: update spoon and shelf

File: assets/urdf/shelf/urdf/shelf.urdf (robot description, URDF)
Before this commit: robot shelf, 1 links, 0 joints
Links:
- link base_link: geometry collision box size=0.002 0.1 0.085; collision box size=0.002 0.1 0.085
