Commit message: update urdf

File: assets/urdf/cup/urdf/cup.urdf (robot description, URDF)
Before this commit: robot cup, 1 links, 0 joints
Links:
- link base_link: mass 0.980227529286016 -> 0.98023

File: assets/urdf/spoon/urdf/spoon.urdf (robot description, URDF)
Before this commit: robot spoon, 1 links, 0 joints
Links:
- link base_link: mass 0.0022598 -> 0.040738

Commit message: sync urdf

File: assets/urdf/cup/urdf/cup.urdf (robot description, URDF)
Before this commit: robot cup, 1 links, 0 joints
Links:
- link base_link: mass 0.98023 -> 0.35723

File: assets/urdf/spoon/urdf/spoon.urdf (robot description, URDF)
Before this commit: robot spoon, 1 links, 0 joints
Links:
- link base_link: mass 0.040738 -> 0.032987

Commit message: sync fix air wall

File: assets/urdf/cup/urdf/cup.urdf (robot description, URDF)
Before this commit: robot cup, 1 links, 0 joints
Links:
- link base_link: mass 0.35723 -> 0.1035; geometry collision box size=0.002 0.1 0.05; collision box size=0.002 0.1 0.05

File: assets/urdf/shelf/urdf/shelf.urdf (robot description, URDF)
Before this commit: robot shelf, 1 links, 0 joints
Links:
- link base_link: geometry collision box size=0.011 0.11 0.07534; collision box size=0.011 0.11 0.07534

Commit message: replace franka to the curi
add docs and asset

File: assets/urdf/cup/urdf/cup.urdf (robot description, URDF)
Before this commit: robot cup3, 1 links, 0 joints
Links:
- link base_link: geometry collision box size=0.002 0.1 0.05; collision box size=0.002 0.1 0.05

File: assets/urdf/shelf/urdf/shelf.urdf (robot description, URDF)
Before this commit: robot shelf, 1 links, 0 joints
Links:
- link base_link: geometry collision box size=0.002 0.1 0.085; collision box size=0.002 0.1 0.085
